Commit message: add ability to have different colored spot models

File: spot_tools_ros/urdf/spot.urdf.xacro (robot description, xacro)
@@ -11,8 +11,11 @@
   <!-- Set to true to enable joints -->
   <xacro:arg name="include_transmissions" default="true" />^M
+  <!-- Set to the accent color you want for spot -->
+  <xacro:arg name="spot_color" default="yellow" />
   <!-- Load Spot -->
   <xacro:load_spot
     arm="$(arg arm)"
     tf_prefix="$(arg tf_prefix)"
+    spot_color="$(arg spot_color)"
     gripperless="$(arg gripperless)"
     include_transmissions="$(arg include_transmissions)" />

File: spot_tools_ros/urdf/spot_macro.xacro (robot description, xacro)
@@ -3,18 +3,22 @@
     <xacro:macro name="load_spot" params="
     arm:=false
+    tf_prefix
+    spot_color:=yellow
     gripperless:=false
     custom_gripper_base_link:=''
-    tf_prefix
     include_transmissions=false">
         <link name="${tf_prefix}body">
             <visual>
                 <geometry>
-                    <mesh filename="package://spot_tools_ros/meshes/base/visual/body.obj" />
-                </geometry>
-            </visual>
-            <collision>
-                <geometry>
-                    <mesh
-                        filename="package://spot_tools_ros/meshes/base/collision/body_collision.obj" />
+                    <mesh filename="package://spot_tools_ros/meshes/visual/spot_${spot_color}/body.obj" />
+                </geometry>
+                <material name="red">
+                    <color rgba="1 0 0 1"/>
+                </material>
+            </visual>
+            <collision>
+                <geometry>
+                    <mesh
+                        filename="package://spot_tools_ros/meshes/collision/body_collision.obj" />
                 </geometry>
             </collision>
@@ -62,5 +66,5 @@
                 <geometry>
                     <mesh
-                        filename="package://spot_tools_ros/meshes/base/visual/front_left_hip.obj" />
+                        filename="package://spot_tools_ros/meshes/visual/spot_${spot_color}/front_left_hip.obj" />
                 </geometry>
             </visual>
@@ -96,11 +100,11 @@
                 <geometry>
                     <mesh
-                        filename="package://spot_tools_ros/meshes/base/visual/front_left_upper_leg.obj" />
-                </geometry>
-            </visual>
-            <collision>
-                <geometry>
-                    <mesh
-                        filename="package://spot_tools_ros/meshes/base/collision/left_upper_leg_collision.obj" />
+                        filename="package://spot_tools_ros/meshes/visual/spot_${spot_color}/front_left_upper_leg.obj" />
+                </geometry>
+            </visual>
+            <collision>
+                <geometry>
+                    <mesh
+                        filename="package://spot_tools_ros/meshes/collision/left_upper_leg_collision.obj" />
                 </geometry>
             </collision>
@@ -136,11 +140,11 @@
                 <geometry>
                     <mesh
-                        filename="package://spot_tools_ros/meshes/base/visual/front_left_lower_leg.obj" />
-                </geometry>
-            </visual>
-            <collision>
-                <geometry>
-                    <mesh
-                        filename="package://spot_tools_ros/meshes/base/collision/left_lower_leg_collision.obj" />
+                        filename="package://spot_tools_ros/meshes/visual/spot_${spot_color}/front_left_lower_leg.obj" />
+                </geometry>
+            </visual>
+            <collision>
+                <geometry>
+                    <mesh
+                        filename="package://spot_tools_ros/meshes/collision/left_lower_leg_collision.obj" />
                 </geometry>
             </collision>
@@ -182,5 +186,5 @@
                 <geometry>
                     <mesh
-                        filename="package://spot_tools_ros/meshes/base/visual/front_right_hip.obj" />
+                        filename="package://spot_tools_ros/meshes/visual/spot_${spot_color}/front_right_hip.obj" />
                 </geometry>
             </visual>
@@ -216,11 +220,11 @@
                 <geometry>
                     <mesh
-                        filename="package://spot_tools_ros/meshes/base/visual/front_right_upper_leg.obj" />
-                </geometry>
-            </visual>
-            <collision>
-                <geometry>
-                    <mesh
-                        filename="package://spot_tools_ros/meshes/base/collision/right_upper_leg_collision.obj" />
+                        filename="package://spot_tools_ros/meshes/visual/spot_${spot_color}/front_right_upper_leg.obj" />
+                </geometry>
+            </visual>
+            <collision>
+                <geometry>
+                    <mesh
+                        filename="package://spot_tools_ros/meshes/collision/right_upper_leg_collision.obj" />
                 </geometry>
             </collision>
@@ -256,11 +260,11 @@
                 <geometry>
                     <mesh
-                        filename="package://spot_tools_ros/meshes/base/visual/front_right_lower_leg.obj" />
-                </geometry>
-            </visual>
-            <collision>
-                <geometry>
-                    <mesh
-                        filename="package://spot_tools_ros/meshes/base/collision/right_lower_leg_collision.obj" />
+                        filename="package://spot_tools_ros/meshes/visual/spot_${spot_color}/front_right_lower_leg.obj" />
+                </geometry>
+            </visual>
+            <collision>
+                <geometry>
+                    <mesh
+                        filename="package://spot_tools_ros/meshes/collision/right_lower_leg_collision.obj" />
                 </geometry>
             </collision>
@@ -302,5 +306,5 @@
                 <geometry>
                     <mesh
-                        filename="package://spot_tools_ros/meshes/base/visual/rear_left_hip.obj" />
+                        filename="package://spot_tools_ros/meshes/visual/spot_${spot_color}/rear_left_hip.obj" />
                 </geometry>
             </visual>
@@ -336,11 +340,11 @@
                 <geometry>
                     <mesh
-                        filename="package://spot_tools_ros/meshes/base/visual/rear_left_upper_leg.obj" />
-                </geometry>
-            </visual>
-            <collision>
-                <geometry>
-                    <mesh
-                        filename="package://spot_tools_ros/meshes/base/collision/left_upper_leg_collision.obj" />
+                        filename="package://spot_tools_ros/meshes/visual/spot_${spot_color}/rear_left_upper_leg.obj" />
+                </geometry>
+            </visual>
+            <collision>
+                <geometry>
+                    <mesh
+                        filename="package://spot_tools_ros/meshes/collision/left_upper_leg_collision.obj" />
                 </geometry>
             </collision>
@@ -376,11 +380,11 @@
                 <geometry>
                     <mesh
-                        filename="package://spot_tools_ros/meshes/base/visual/rear_left_lower_leg.obj" />
-                </geometry>
-            </visual>
-            <collision>
-                <geometry>
-                    <mesh
-                        filename="package://spot_tools_ros/meshes/base/collision/left_lower_leg_collision.obj" />
+                        filename="package://spot_tools_ros/meshes/visual/spot_${spot_color}/rear_left_lower_leg.obj" />
+                </geometry>
+            </visual>
+            <collision>
+                <geometry>
+                    <mesh
+                        filename="package://spot_tools_ros/meshes/collision/left_lower_leg_collision.obj" />
                 </geometry>
             </collision>
@@ -422,5 +426,5 @@
                 <geometry>
                     <mesh
-                        filename="package://spot_tools_ros/meshes/base/visual/rear_right_hip.obj" />
+                        filename="package://spot_tools_ros/meshes/visual/spot_${spot_color}/rear_right_hip.obj" />
                 </geometry>
             </visual>
@@ -456,11 +460,11 @@
                 <geometry>
                     <mesh
-                        filename="package://spot_tools_ros/meshes/base/visual/rear_right_upper_leg.obj" />
-                </geometry>
-            </visual>
-            <collision>
-                <geometry>
-                    <mesh
-                        filename="package://spot_tools_ros/meshes/base/collision/right_upper_leg_collision.obj" />
+                        filename="package://spot_tools_ros/meshes/visual/spot_${spot_color}/rear_right_upper_leg.obj" />
+                </geometry>
+            </visual>
+            <collision>
+                <geometry>
+                    <mesh
+                        filename="package://spot_tools_ros/meshes/collision/right_upper_leg_collision.obj" />
                 </geometry>
             </collision>
@@ -496,11 +500,11 @@
                 <geometry>
                     <mesh
-                        filename="package://spot_tools_ros/meshes/base/visual/rear_right_lower_leg.obj" />
-                </geometry>
-            </visual>
-            <collision>
-                <geometry>
-                    <mesh
-                        filename="package://spot_tools_ros/meshes/base/collision/right_lower_leg_collision.obj" />
+                        filename="package://spot_tools_ros/meshes/visual/spot_${spot_color}/rear_right_lower_leg.obj" />
+                </geometry>
+            </visual>
+            <collision>
+                <geometry>
+                    <mesh
+                        filename="package://spot_tools_ros/meshes/collision/right_lower_leg_collision.obj" />
                 </geometry>
             </collision>
@@ -544,5 +548,5 @@
         <xacro:if value="${arm}">
             <xacro:include filename="$(find spot_tools_ros)/urdf/spot_arm_macro.urdf" />
-            <xacro:load_arm tf_prefix="${tf_prefix}" gripperless="${gripperless}" custom_gripper_base_link="${custom_gripper_base_link}" />
+            <xacro:load_arm tf_prefix="${tf_prefix}" spot_color="spot_${spot_color}" gripperless="${gripperless}" custom_gripper_base_link="${custom_gripper_base_link}" />
         </xacro:if>
     </xacro:macro>

Commit message: allow extending with macro

File: spot_tools_ros/urdf/spot.urdf.xacro (robot description, xacro)
@@ -10,7 +10,7 @@
   <xacro:arg name="gripperless" default="false" />
   <!-- Set to true to enable joints -->
-  <xacro:arg name="include_transmissions" default="true" />^M
+  <xacro:arg name="include_transmissions" default="true"/>
   <!-- Set to the accent color you want for spot -->
-  <xacro:arg name="spot_color" default="yellow" />
+  <xacro:arg name="spot_color" default="yellow"/>
   <!-- Load Spot -->
   <xacro:load_spot
@@ -19,4 +19,8 @@
     spot_color="$(arg spot_color)"
     gripperless="$(arg gripperless)"
-    include_transmissions="$(arg include_transmissions)" />
+    include_transmissions="$(arg include_transmissions)"/>
+  <!-- Optional custom includes. -->
+  <xacro:arg name="extras_urdf" default="$(find spot_tools_ros)/urdf/empty.urdf.xacro"/>
+  <xacro:include filename="$(arg extras_urdf)"/>
+  <xacro:load_extras tf_prefix="$(arg tf_prefix)"/>
 </robot>

File: spot_tools_ros/urdf/spot_macro.xacro (robot description, xacro)
@@ -542,7 +542,4 @@
                     </transmission>
         </xacro:if>
-        <!-- Optional custom includes. -->
-        <xacro:property name="default_empty_urdf" value="$(find spot_tools_ros)/urdf/empty.urdf" />
-        <xacro:include filename="$(optenv SPOT_URDF_EXTRAS ${default_empty_urdf})" />
         <!-- Include Arm if necessary-->
         <xacro:if value="${arm}">
